File: hardware/Walle_E_ESP32_S3_Node_v2.kicad_sch (KiCad schematic)
At the start: 46 parts, among them J1 Voltage01_ZMPT101B, J10 Conn_01x22_Pin, J11 Conn_01x22_Pin, J12 Conn_01x08_Pin, J13 Conn_01x08_Pin, J14 Diff_Pressure_Sens LWLP5000, J2 CurrentSens01_ACS712_5A, J4 CurrentSens03_ACS712_5A, J5 Conn_01x04_Pin, J6 +5VdcSupply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

Commit message: Thickness improve in AC current sensor input AC line
Parts:
- PS2: footprint RAC05-05SK_schematic:CONV_RAC05-05SK -> RAC05-05SK:CONV_RAC05-05SK
- U1: footprint ESP32-S3-DEVKITC-1-N16R8V footprint:XCVR_ESP32-S3-DEVKITC-1-N16R8V -> ESP32-S3-DEVKITC-1-N16R8V:XCVR_ESP32-S3-DEVKITC-1-N16R8V
- U2: footprint RA-02_LORA footprint:MODULE_RA-02_LORA -> RA-02_LORA:MODULE_RA-02_LORA
Changed lines of the file:
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@@
 			)
 		)
-		(property "Footprint" "ESP32-S3-DEVKITC-1-N16R8V footprint:XCVR_ESP32-S3-DEVKITC-1-N16R8V"
+		(property "Footprint" "ESP32-S3-DEVKITC-1-N16R8V:XCVR_ESP32-S3-DEVKITC-1-N16R8V"
 			(at 200.66 73.66 0)
 			(effects
@@
 			)
 		)
-		(property "Footprint" "RAC05-05SK_schematic:CONV_RAC05-05SK"
+		(property "Footprint" "RAC05-05SK:CONV_RAC05-05SK"
 			(at 142.24 27.94 0)
 			(effects
@@
 			)
 		)
-		(property "Footprint" "RA-02_LORA footprint:MODULE_RA-02_LORA"
+		(property "Footprint" "RA-02_LORA:MODULE_RA-02_LORA"
 			(at 54.61 184.15 0)
 			(effects
